File: SBC Circuit/SBC Circuit.kicad_pcb (KiCad board)
At the start: 2 copper layers, 0 parts

Commit message: Grouped footprints on PCB
Parts:
- added C1: 4.7u, Capacitor_THT:CP_Radial_D4.0mm_P2.00mm, F.Cu at (-500.9, 239.5)
- added C10: 0.1u, Capacitor_THT:CP_Box_L5.50mm_W4.00mm_P2.50mm_NonPolarized, F.Cu at (-527.8, -29.9)
- added C11: 1u, Capacitor_THT:CP_Box_L5.50mm_W4.00mm_P2.50mm_NonPolarized, F.Cu at (-527.5, -40.9)
- added C12: 0.1u, Capacitor_THT:CP_Box_L5.50mm_W4.00mm_P2.50mm_NonPolarized, F.Cu at (-512.3, -31.4)
- added C13: 1u, Capacitor_THT:CP_Box_L5.50mm_W4.00mm_P2.50mm_NonPolarized, F.Cu at (-512.5, -40.9)
- added C14: 0.1u, Capacitor_THT:CP_Box_L5.50mm_W4.00mm_P2.50mm_NonPolarized, F.Cu at (-495.0, -41.9)
- added C15: 1u, Capacitor_THT:CP_Box_L5.50mm_W4.00mm_P2.50mm_NonPolarized, F.Cu at (-495.3, -30.9)
- added C16: .1u, Capacitor_THT:CP_Box_L5.50mm_W4.00mm_P2.50mm_NonPolarized, F.Cu at (-701.5, 13.9)
- added C17: 1u, Capacitor_THT:CP_Box_L5.50mm_W4.00mm_P2.50mm_NonPolarized, F.Cu at (-687.5, 14.9)
- added C18: .1u, Capacitor_THT:CP_Box_L5.50mm_W4.00mm_P2.50mm_NonPolarized, F.Cu at (-394.9, 91.4)
- added C19: 1u, Capacitor_THT:CP_Box_L5.50mm_W4.00mm_P2.50mm_NonPolarized, F.Cu at (-386.7, 91.4)
- added C2: 4.7u, Capacitor_THT:CP_Radial_D4.0mm_P2.00mm, F.Cu at (-457.5, 255.0)
- added C20: .1u, Capacitor_THT:CP_Box_L5.50mm_W4.00mm_P2.50mm_NonPolarized, F.Cu at (-350.9, 91.4)
- added C21: 1u, Capacitor_THT:CP_Box_L5.50mm_W4.00mm_P2.50mm_NonPolarized, F.Cu at (-359.9, 92.4)
- added C22: .1u, Capacitor_THT:CP_Box_L5.50mm_W4.00mm_P2.50mm_NonPolarized, F.Cu at (-404.9, -24.8)
- added C23: 1u, Capacitor_THT:CP_Box_L5.50mm_W4.00mm_P2.50mm_NonPolarized, F.Cu at (-414.4, -23.8)
- added C24: .1u, Capacitor_THT:CP_Box_L5.50mm_W4.00mm_P2.50mm_NonPolarized, F.Cu at (-357.6, -24.8)
- added C25: 1u, Capacitor_THT:CP_Box_L5.50mm_W4.00mm_P2.50mm_NonPolarized, F.Cu at (-366.1, -24.8)
- added C26: 0.1u, Capacitor_THT:CP_Box_L5.50mm_W4.00mm_P2.50mm_NonPolarized, F.Cu at (-678.1, 206.0)
- added C27: 1u, Capacitor_THT:CP_Box_L5.50mm_W4.00mm_P2.50mm_NonPolarized, F.Cu at (-670.6, 206.0)
- added C28: .1u, Capacitor_THT:CP_Box_L5.50mm_W4.00mm_P2.50mm_NonPolarized, F.Cu at (-703.9, 207.5)
- added C29: .1u, Capacitor_THT:CP_Box_L5.50mm_W4.00mm_P2.50mm_NonPolarized, F.Cu at (-694.1, 207.5)
- added C3: 4.7u, Capacitor_THT:CP_Radial_D4.0mm_P2.00mm, F.Cu at (-595.0, 252.5)
- added C30: 47p, Capacitor_THT:CP_Box_L5.50mm_W4.00mm_P2.50mm_NonPolarized, F.Cu at (-696.9, 186.0)
- added C31: 47p, Capacitor_THT:CP_Box_L5.50mm_W4.00mm_P2.50mm_NonPolarized, F.Cu at (-707.9, 187.0)
- added C4: 10n, Capacitor_THT:CP_Box_L5.50mm_W4.00mm_P2.50mm_NonPolarized, F.Cu at (-573.2, 304.0)
- added C5: 0.1u, Capacitor_THT:CP_Box_L5.50mm_W4.00mm_P2.50mm_NonPolarized, F.Cu at (-457.8, 100.8)
- added C6: 0.1u, Capacitor_THT:CP_Box_L5.50mm_W4.00mm_P2.50mm_NonPolarized, F.Cu at (-525.0, 130.0)
- added C7: 1u, Capacitor_THT:CP_Box_L5.50mm_W4.00mm_P2.50mm_NonPolarized, F.Cu at (-525.0, 140.0)
- added C8: 0.1u, Capacitor_THT:CP_Box_L5.50mm_W4.00mm_P2.50mm_NonPolarized, F.Cu at (-483.2, 131.0)
- added C9: 1u, Capacitor_THT:CP_Box_L5.50mm_W4.00mm_P2.50mm_NonPolarized, F.Cu at (-483.0, 142.0)
- added D1: 1N4001, Diode_THT:D_DO-41_SOD81_P5.08mm_Vertical_KathodeUp, F.Cu at (-578.8, 260.0)
- added D2: 1N4001, Diode_THT:D_DO-41_SOD81_P5.08mm_Vertical_KathodeUp, F.Cu at (-458.8, 248.0)
- added D3: LED, LED_THT:LED_D5.0mm, F.Cu at (-509.0, 226.5)
- added D4: LED, LED_THT:LED_D5.0mm, F.Cu at (-458.5, 261.5)
- added D5: LED, LED_THT:LED_D5.0mm, F.Cu at (-679.6, 179.0)
- added D6: LED, LED_THT:LED_D5.0mm, F.Cu at (-672.1, 179.0)
- added F1: 250mA Fuse, Fuse:Fuseholder_Clip-5x20mm_Bel_FC-203-22_Lateral_P17.80x5.00mm_D1.17mm_Horizontal, F.Cu at (-582.4, 249.0)
- added F2: 250mA Fuse, Fuse:Fuseholder_Clip-5x20mm_Bel_FC-203-22_Lateral_P17.80x5.00mm_D1.17mm_Horizontal, F.Cu at (-591.9, 291.0)
- added FB1: FerriteBead, Capacitor_THT:C_Axial_L3.8mm_D2.6mm_P10.00mm_Horizontal, F.Cu at (-583.5, 279.0)
- added J1: USB_B, Connector_USB:USB_B_OST_USB-B1HSxx_Horizontal, F.Cu at (-569.1, 286.2)
- added J10: Conn_01x02_Pin, Connector_PinHeader_2.54mm:PinHeader_1x02_P2.54mm_Vertical, F.Cu at (-669.8, 188.8)
- added J11: Conn_01x02_Pin, Connector_PinHeader_2.54mm:PinHeader_1x02_P2.54mm_Vertical, F.Cu at (-663.6, 188.5)
- added J12: Conn_01x02_Pin, Connector_PinHeader_2.54mm:PinHeader_1x02_P2.54mm_Vertical, F.Cu at (-659.0, 188.5)
- added J2: Conn_01x02_Pin, Connector_PinHeader_2.54mm:PinHeader_1x02_P2.54mm_Vertical, F.Cu at (-559.5, 250.2)
- added J3: Conn_01x06_Pin, Connector_PinHeader_2.54mm:PinHeader_1x06_P2.54mm_Vertical, F.Cu at (-534.6, -19.0)
- added J4: Conn_01x06_Pin, Connector_PinHeader_2.54mm:PinHeader_1x06_P2.54mm_Vertical, F.Cu at (-653.0, 182.2)
- added J5: Conn_01x03_Pin, Connector_PinHeader_2.54mm:PinHeader_1x03_P2.54mm_Vertical, F.Cu at (-684.4, 72.7)
- added J6: Conn_01x08_Pin, Connector_PinHeader_2.54mm:PinHeader_1x08_P2.54mm_Vertical, F.Cu at (-695.4, 49.2)
- added J7: Conn_01x06_Pin, Connector_PinHeader_2.54mm:PinHeader_1x06_P2.54mm_Vertical, F.Cu at (-685.4, 43.8)
- added J8: Conn_01x02_Pin, Connector_PinHeader_2.54mm:PinHeader_1x02_P2.54mm_Vertical, F.Cu at (-684.8, 188.5)
- added J9: Conn_01x02_Pin, Connector_PinHeader_2.54mm:PinHeader_1x02_P2.54mm_Vertical, F.Cu at (-676.3, 188.8)
- added Q1: AOI21357, Package_TO_SOT_THT:TO-220-3_Vertical, F.Cu at (-491.5, 222.9)
- added Q2: AOI21357, Package_TO_SOT_THT:TO-220-3_Vertical, F.Cu at (-469.1, 248.0)
- added R1: 1M, Resistor_THT:R_Axial_DIN0204_L3.6mm_D1.6mm_P2.54mm_Vertical, F.Cu at (-589.7, 251.5)
- added R10: 220, Resistor_THT:R_Axial_DIN0204_L3.6mm_D1.6mm_P2.54mm_Vertical, F.Cu at (-696.2, 175.0)
- added R2: 10k, Resistor_THT:R_Axial_DIN0204_L3.6mm_D1.6mm_P2.54mm_Vertical, F.Cu at (-531.0, 118.0)
- added R3: 10k, Resistor_THT:R_Axial_DIN0204_L3.6mm_D1.6mm_P2.54mm_Vertical, F.Cu at (-474.8, 89.2)
- added R4: 10k, Resistor_THT:R_Axial_DIN0204_L3.6mm_D1.6mm_P2.54mm_Vertical, F.Cu at (-468.2, 91.2)
- added R5: 5.6k, Resistor_THT:R_Axial_DIN0204_L3.6mm_D1.6mm_P2.54mm_Vertical, F.Cu at (-653.1, 206.0)
- added R6: 10k, Resistor_THT:R_Axial_DIN0204_L3.6mm_D1.6mm_P2.54mm_Vertical, F.Cu at (-647.8, 206.0)
- added R7: 470, Resistor_THT:R_Axial_DIN0204_L3.6mm_D1.6mm_P2.54mm_Vertical, F.Cu at (-492.1, 240.0)
- added R8: 220, Resistor_THT:R_Axial_DIN0204_L3.6mm_D1.6mm_P2.54mm_Vertical, F.Cu at (-469.7, 262.5)
- added R9: 220, Resistor_THT:R_Axial_DIN0204_L3.6mm_D1.6mm_P2.54mm_Vertical, F.Cu at (-695.6, 168.0)
- added SW1: RESET, Button_Switch_THT:SW_PUSH_6mm, F.Cu at (-471.0, 98.5)
- added TP1: 5V TEST, TestPoint:TestPoint_Keystone_5000-5004_Miniature, F.Cu at (-496.9, 232.0)
- added TP2: 3V TEST, TestPoint:TestPoint_Keystone_5000-5004_Miniature, F.Cu at (-474.5, 256.0)
- added TP3: ~{HLT}/~{RST}, TestPoint:TestPoint_Keystone_5000-5004_Miniature, F.Cu at (-477.8, 104.2)
- added TP4: VBUS SENSE, TestPoint:TestPoint_Keystone_5000-5004_Miniature, F.Cu at (-641.0, 188.3)
- added U1: MC68000FN, Package_LCC:PLCC-68_THT-Socket, F.Cu at (-506.3, 122.3)
- added U10: FT230XS, Package_SO:SSOP-16_3.9x4.9mm_P0.635mm, F.Cu at (-646.6, 188.0)
- added U11: MC34064P, Package_TO_SOT_THT:TO-92_Inline, F.Cu at (-469.0, 109.6)
- added U2: XC9572XL, Package_LCC:PLCC-44_THT-Socket, F.Cu at (-505.6, -18.1)
- added U3: 68681, Package_DIP:DIP-40_W15.24mm_Socket, F.Cu at (-663.0, 31.1)
- added U4: MCM6206CP, Package_DIP:DIP-28_W7.62mm_Socket, F.Cu at (-382.1, 101.4)
- added U5: MCM6206CP, Package_DIP:DIP-28_W7.62mm_Socket, F.Cu at (-359.7, 102.4)
- added U6: 28C256, Package_DIP:DIP-28_W15.24mm_Socket, F.Cu at (-413.1, -15.0)
- added U7: 28C256, Package_DIP:DIP-28_W15.24mm_Socket, F.Cu at (-368.1, -15.0)
- added U8: LM7805_TO220, Package_TO_SOT_THT:TO-220-3_Vertical, F.Cu at (-491.5, 232.0)
- added U9: LD1117AV33, Package_TO_SOT_THT:TO-220-3_Vertical, F.Cu at (-469.1, 256.0)
- added X1: SG-531, Oscillator:Oscillator_SeikoEpson_SG-8002DC, F.Cu at (-547.6, 128.0)
- added X2: EC11, Oscillator:Oscillator_DIP-8, F.Cu at (-659.4, 20.4)
