File: SBC Circuit/SBC Circuit.kicad_pcb (KiCad board)
At the start: 2 copper layers, 82 parts, among them J1 USB_B, J10 Conn_01x02_Pin, J11 Conn_01x02_Pin, J12 Conn_01x02_Pin, J2 Conn_01x02_Pin, J3 Conn_01x06_Pin, J4 Conn_01x06_Pin, J5 Conn_01x03_Pin, J6 Conn_01x08_Pin, J7 Conn_01x06_Pin, J8 Conn_01x02_Pin, J9 Conn_01x02_Pin, Q1 AOI21357, Q2 AOI21357, SW1 RESET, U1 MC68000FN, U10 FT230XS, U11 MC34064P, U2 XC9572XL, U3 68681, U4 MCM6206CP, U5 MCM6206CP, U6 28C256, U7 28C256, U8 LM7805_TO220, U9 LD1117AV33, X1 SG-531, X2 EC11

Commit message: Fix intersheet bus issues
Connections:
- net /addr15 renamed addr15
- net /addr16 renamed addr16
- net /addr17 renamed addr17
- net /addr18 renamed addr18
- net /addr19 renamed addr19
- net /addr20 renamed addr20
- net /addr21 renamed addr21
- net /addr22 renamed addr22
- U1 pad 1: /data4 -> data4
- U1 pad 2: /data3 -> data3
- U1 pad 3: /data2 -> data2
- U1 pad 32: /addr0 -> addr0
- U1 pad 33: /addr1 -> addr1
- U1 pad 34: /addr2 -> addr2
- U1 pad 35: /addr3 -> addr3
- U1 pad 36: /addr4 -> addr4
- U1 pad 37: /addr5 -> addr5
- U1 pad 38: /addr6 -> addr6
- U1 pad 39: /addr7 -> addr7
- U1 pad 4: /data1 -> data1
- U1 pad 40: /addr8 -> addr8
- U1 pad 41: /addr9 -> addr9
- U1 pad 42: /addr10 -> addr10
- U1 pad 43: /addr11 -> addr11
- U1 pad 44: /addr12 -> addr12
- U1 pad 45: /addr13 -> addr13
- U1 pad 46: /addr14 -> addr14
- U1 pad 5: /data0 -> data0
- U1 pad 58: /data15 -> data15
- U1 pad 59: /data14 -> data14
- U1 pad 60: /data13 -> data13
- U1 pad 61: /data12 -> data12
- U1 pad 62: /data11 -> data11
- U1 pad 63: /data10 -> data10
- U1 pad 64: /data9 -> data9
- U1 pad 65: /data8 -> data8
- U1 pad 66: /data7 -> data7
- U1 pad 67: /data6 -> data6
- U1 pad 68: /data5 -> data5
- U2 pad 43: unconnected-(U2-P43-Pad43) -> oe
- U2 pad 44: unconnected-(U2-P44-Pad44) -> we
- U3 pad 1: /Memory+Peripheral/addr0 -> addr0
- U3 pad 16: /Memory+Peripheral/data1 -> data1
- U3 pad 17: /Memory+Peripheral/data3 -> data3
- U3 pad 18: /Memory+Peripheral/data5 -> data5
- U3 pad 19: /Memory+Peripheral/data7 -> data7
- U3 pad 22: /Memory+Peripheral/data6 -> data6
- U3 pad 23: /Memory+Peripheral/data4 -> data4
- U3 pad 24: /Memory+Peripheral/data2 -> data2
- U3 pad 25: /Memory+Peripheral/data0 -> data0
- U3 pad 3: /Memory+Peripheral/addr1 -> addr1
- U3 pad 5: /Memory+Peripheral/addr2 -> addr2
- U3 pad 6: /Memory+Peripheral/addr3 -> addr3
- U4 pad 1: /Memory+Peripheral/addr14 -> addr14
- U4 pad 10: /Memory+Peripheral/addr0 -> addr0
- U4 pad 11: /Memory+Peripheral/data0 -> data0
- U4 pad 12: /Memory+Peripheral/data1 -> data1
- U4 pad 13: /Memory+Peripheral/data2 -> data2
- U4 pad 15: /Memory+Peripheral/data3 -> data3
- U4 pad 16: /Memory+Peripheral/data4 -> data4
- U4 pad 17: /Memory+Peripheral/data5 -> data5
- U4 pad 18: /Memory+Peripheral/data6 -> data6
- U4 pad 19: /Memory+Peripheral/data7 -> data7
- U4 pad 2: /Memory+Peripheral/addr12 -> addr12
- U4 pad 21: /Memory+Peripheral/addr10 -> addr10
- U4 pad 22: /Memory+Peripheral/oe -> oe
- U4 pad 23: /Memory+Peripheral/addr11 -> addr11
- U4 pad 24: /Memory+Peripheral/addr9 -> addr9
- U4 pad 25: /Memory+Peripheral/addr8 -> addr8
- U4 pad 26: /Memory+Peripheral/addr13 -> addr13
- U4 pad 27: /Memory+Peripheral/we -> we
- U4 pad 3: /Memory+Peripheral/addr7 -> addr7
- U4 pad 4: /Memory+Peripheral/addr6 -> addr6
- U4 pad 5: /Memory+Peripheral/addr5 -> addr5
- U4 pad 6: /Memory+Peripheral/addr4 -> addr4
- U4 pad 7: /Memory+Peripheral/addr3 -> addr3
- U4 pad 8: /Memory+Peripheral/addr2 -> addr2
- U4 pad 9: /Memory+Peripheral/addr1 -> addr1
- U5 pad 1: /Memory+Peripheral/addr14 -> addr14
- U5 pad 10: /Memory+Peripheral/addr0 -> addr0
- U5 pad 11: /Memory+Peripheral/data8 -> data8
- U5 pad 12: /Memory+Peripheral/data9 -> data9
- U5 pad 13: /Memory+Peripheral/data10 -> data10
- U5 pad 15: /Memory+Peripheral/data11 -> data11
- U5 pad 16: /Memory+Peripheral/data12 -> data12
- U5 pad 17: /Memory+Peripheral/data13 -> data13
- U5 pad 18: /Memory+Peripheral/data14 -> data14
- U5 pad 19: /Memory+Peripheral/data15 -> data15
- U5 pad 2: /Memory+Peripheral/addr12 -> addr12
- U5 pad 21: /Memory+Peripheral/addr10 -> addr10
- U5 pad 22: /Memory+Peripheral/oe -> oe
- U5 pad 23: /Memory+Peripheral/addr11 -> addr11
- U5 pad 24: /Memory+Peripheral/addr9 -> addr9
- U5 pad 25: /Memory+Peripheral/addr8 -> addr8
- U5 pad 26: /Memory+Peripheral/addr13 -> addr13
- U5 pad 27: /Memory+Peripheral/we -> we
- U5 pad 3: /Memory+Peripheral/addr7 -> addr7
- U5 pad 4: /Memory+Peripheral/addr6 -> addr6
- U5 pad 5: /Memory+Peripheral/addr5 -> addr5
- U5 pad 6: /Memory+Peripheral/addr4 -> addr4
- U5 pad 7: /Memory+Peripheral/addr3 -> addr3
- U5 pad 8: /Memory+Peripheral/addr2 -> addr2
- U5 pad 9: /Memory+Peripheral/addr1 -> addr1
- U6 pad 1: /Memory+Peripheral/addr14 -> addr14
- U6 pad 10: /Memory+Peripheral/addr0 -> addr0
- U6 pad 11: /Memory+Peripheral/data0 -> data0
- U6 pad 12: /Memory+Peripheral/data1 -> data1
- U6 pad 13: /Memory+Peripheral/data2 -> data2
- U6 pad 15: /Memory+Peripheral/data3 -> data3
- U6 pad 16: /Memory+Peripheral/data4 -> data4
- U6 pad 17: /Memory+Peripheral/data5 -> data5
- U6 pad 18: /Memory+Peripheral/data6 -> data6
- U6 pad 19: /Memory+Peripheral/data7 -> data7
- U6 pad 2: /Memory+Peripheral/addr12 -> addr12
- U6 pad 21: /Memory+Peripheral/addr10 -> addr10
- U6 pad 22: /Memory+Peripheral/oe -> oe
- U6 pad 23: /Memory+Peripheral/addr11 -> addr11
- U6 pad 24: /Memory+Peripheral/addr9 -> addr9
- U6 pad 25: /Memory+Peripheral/addr8 -> addr8
- U6 pad 26: /Memory+Peripheral/addr13 -> addr13
- U6 pad 27: /Memory+Peripheral/we -> we
- U6 pad 3: /Memory+Peripheral/addr7 -> addr7
- U6 pad 4: /Memory+Peripheral/addr6 -> addr6
- U6 pad 5: /Memory+Peripheral/addr5 -> addr5
- U6 pad 6: /Memory+Peripheral/addr4 -> addr4
- U6 pad 7: /Memory+Peripheral/addr3 -> addr3
- U6 pad 8: /Memory+Peripheral/addr2 -> addr2
- U6 pad 9: /Memory+Peripheral/addr1 -> addr1
- U7 pad 1: /Memory+Peripheral/addr14 -> addr14
- U7 pad 10: /Memory+Peripheral/addr0 -> addr0
- U7 pad 11: /Memory+Peripheral/data8 -> data8
- U7 pad 12: /Memory+Peripheral/data9 -> data9
- U7 pad 13: /Memory+Peripheral/data10 -> data10
- U7 pad 15: /Memory+Peripheral/data11 -> data11
- U7 pad 16: /Memory+Peripheral/data12 -> data12
- U7 pad 17: /Memory+Peripheral/data13 -> data13
- U7 pad 18: /Memory+Peripheral/data14 -> data14
- U7 pad 19: /Memory+Peripheral/data15 -> data15
- U7 pad 2: /Memory+Peripheral/addr12 -> addr12
- U7 pad 21: /Memory+Peripheral/addr10 -> addr10
- U7 pad 22: /Memory+Peripheral/oe -> oe
- U7 pad 23: /Memory+Peripheral/addr11 -> addr11
- U7 pad 24: /Memory+Peripheral/addr9 -> addr9
- U7 pad 25: /Memory+Peripheral/addr8 -> addr8
- U7 pad 26: /Memory+Peripheral/addr13 -> addr13
- U7 pad 27: /Memory+Peripheral/we -> we
- U7 pad 3: /Memory+Peripheral/addr7 -> addr7
- U7 pad 4: /Memory+Peripheral/addr6 -> addr6
- U7 pad 5: /Memory+Peripheral/addr5 -> addr5
- U7 pad 6: /Memory+Peripheral/addr4 -> addr4
- U7 pad 7: /Memory+Peripheral/addr3 -> addr3
- U7 pad 8: /Memory+Peripheral/addr2 -> addr2
- U7 pad 9: /Memory+Peripheral/addr1 -> addr1

Commit message: PCB CPLD to MPU lines wired
Parts:
- removed R2: 10k, Resistor_THT:R_Axial_DIN0204_L3.6mm_D1.6mm_P2.54mm_Vertical
- C10, C11, C12, C13, C14, C15, C16, C17, C18, C19, C20, C21, C22, C23, C24, C25, C26, C27, C28, C29, C30, C31, C4, C5, C6, C7, C8, C9: footprint Capacitor_THT:CP_Box_L5.50mm_W4.00mm_P2.50mm_NonPolarized -> Capacitor_THT:CP_Disc_L5.50mm_W4.00mm_P2.50mm_NonPolarized
- moved C11 154.4 mm to (-515.0, 113.0), turned to -90 degrees
- moved C10 144.0 mm to (-510.5, 113.0), turned to -90 degrees
- moved C14 142.4 mm to (-494.5, 100.5)
- moved C15 135.9 mm to (-494.5, 105.0)
- moved C13 126.1 mm to (-502.0, 84.8), turned to 90 degrees
- moved J3 118.3 mm to (-524.5, 98.9)
- moved C12 117.1 mm to (-497.5, 84.8), turned to 90 degrees
- moved U2 110.7 mm to (-507.5, 92.5)
- moved C5 86.0 mm to (-531.0, 145.8), turned to -90 degrees
- moved R4 85.4 mm to (-536.0, 143.3), turned to -90 degrees
- moved R3 83.4 mm to (-539.8, 141.5), turned to 180 degrees
- moved U11 80.7 mm to (-541.0, 146.0), turned to 180 degrees
- moved SW1 79.0 mm to (-542.5, 132.0), turned to -90 degrees
- moved TP3 73.8 mm to (-536.0, 149.5)
- moved X1 17.4 mm to (-531.6, 121.1)
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Connections:
- U1 pad 12: /n0 -> +5V
- U1 pad 13: /n0 -> +5V
- U1 pad 23: /n0 -> +5V
- U2 pad 1: /ipl0 -> duart_irq
- U2 pad 11: /lds -> unconnected-(U2-P11-Pad11)
- U2 pad 12: /rw -> /berr
- U2 pad 13: /dtack -> /ipl2
- U2 pad 14: /berr -> /dtack
- U2 pad 18: duart_cs -> /lds
- U2 pad 19: duart_iack -> /rw
- U2 pad 2: /ipl1 -> duart_iack
- U2 pad 20: duart_dtack -> /uds
- U2 pad 22: duart_irq -> /as
- U2 pad 24: addr15 -> /ipl1
- U2 pad 25: addr16 -> /fc2
- U2 pad 26: addr17 -> /ipl0
- U2 pad 27: addr18 -> /fc0
- U2 pad 28: addr19 -> /fc1
- U2 pad 29: addr20 -> addr21
- U2 pad 3: /ipl2 -> duart_cs
- U2 pad 33: addr21 -> addr20
- U2 pad 35: raml_cs -> addr18
- U2 pad 36: ramh_cs -> addr19
- U2 pad 37: roml_cs -> addr16
- U2 pad 38: romh_cs -> addr17
- U2 pad 39: hlt_rst -> addr15
- U2 pad 4: /fc0 -> duart_dtack
- U2 pad 42: unconnected-(U2-P42/GTS1-Pad42) -> hlt_rst
- U2 pad 6: /fc1 -> romh_cs
- U2 pad 7: /fc2 -> roml_cs
- U2 pad 8: /as -> ramh_cs
- U2 pad 9: /uds -> raml_cs
Routing:
- net +5V: track 0.00 -> 63.0 mm
- net +3.3V: track 0.00 -> 60.5 mm
- net addr15: track 0.00 -> 58.8 mm
- net addr17: track 0.00 -> 54.9 mm
- net clk: track 0.00 -> 52.3 mm
- net addr16: track 0.00 -> 52.0 mm
- net /berr: track 0.00 -> 51.2 mm
- net addr19: track 0.00 -> 48.5 mm
- net /ipl2: track 0.00 -> 47.2 mm
- net /fc1: track 0.00 -> 46.8 mm
- net /fc0: track 0.00 -> 45.7 mm
- net addr18: track 0.00 -> 45.6 mm
- net /fc2: track 0.00 -> 44.7 mm
- net /ipl0: track 0.00 -> 44.7 mm
- net /ipl1: track 0.00 -> 43.3 mm
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Other:
- board outline added: 108.5 x 98.5 mm

Commit message: Wire reset circuit
Parts:
- moved D3 142.7 mm to (-636.0, 291.5)
- moved R7 142.7 mm to (-619.1, 305.0)
- moved U8 142.7 mm to (-618.5, 297.0)
- moved C1 142.7 mm to (-627.9, 304.5)
- moved Q1 142.7 mm to (-618.5, 288.9)
- moved TP1 141.0 mm to (-627.0, 286.5)
- moved J1 20.4 mm to (-581.1, 302.8)
- moved FB1 16.9 mm to (-592.9, 293.0), turned to -90 degrees
- moved F2 16.8 mm to (-575.1, 290.5), turned to 180 degrees
- moved C4 12.3 mm to (-585.5, 302.8), turned to 90 degrees
- moved SW1 11.8 mm to (-535.5, 141.5)
- moved TP3 11.0 mm to (-525.0, 149.5)
- moved U11 10.8 mm to (-530.4, 144.0), turned to -90 degrees
- moved R3 8.73 mm to (-533.0, 136.0), turned to -90 degrees
- moved C5 7.21 mm to (-525.0, 141.8)
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Routing:
- net hlt_rst: track 3.59 -> 27.2 mm
- net /Power+IO/n3: track 0.00 -> 20.4 mm
- net /n6: track 0.00 -> 12.2 mm
- net +5V: track 63.0 -> 74.4 mm
- net /Power+IO/n4: track 0.00 -> 2.50 mm
Other:
- board size 108.5 x 98.5 mm -> 155.5 x 98.5 mm

Commit message: Wire fuses and USB jack
Parts:
- moved J1 150.6 mm to (-610.5, 155.0), turned to 180 degrees
- moved C4 149.2 mm to (-606.1, 155.0), turned to -90 degrees
- moved Q1 142.2 mm to (-499.6, 210.9)
- moved D3 139.5 mm to (-516.5, 219.4)
- moved C1 139.5 mm to (-508.5, 232.4)
- moved R7 139.5 mm to (-499.7, 232.9)
- moved TP1 139.5 mm to (-507.5, 214.4)
- moved U8 139.5 mm to (-499.0, 224.9)
- moved FB1 133.4 mm to (-598.7, 159.8), turned to 90 degrees
- moved F2 127.0 mm to (-611.1, 168.7), turned to 0 degrees
- moved D1 94.5 mm to (-554.5, 168.7), turned to -90 degrees
- moved F1 80.3 mm to (-582.8, 168.7)
- moved J2 73.0 mm to (-549.0, 178.0), turned to 90 degrees
Routing:
- net /Power+IO/n2: track 0.00 -> 10.5 mm
- net /Power+IO/n4: track 2.50 -> 11.1 mm
- net /Power+IO/n1: track 0.00 -> 7.26 mm
- net /Power+IO/n3: track 20.4 -> 25.8 mm
Other:
- board size 155.5 x 98.5 mm -> 185.3 x 118.5 mm

Commit message: Wire Serial
Parts:
- removed the C28 at (-703.9, 207.5)
- removed J10, J11, J12: Conn_01x02_Pin, Connector_PinHeader_2.54mm:PinHeader_1x02_P2.54mm_Vertical
- J9: value Conn_01x02_Pin -> Conn_02x04_Odd_Even; footprint Connector_PinHeader_2.54mm:PinHeader_1x02_P2.54mm_Vertical -> Connector_PinHeader_2.54mm:PinHeader_2x04_P2.54mm_Vertical
- moved C30 132.3 mm to (-579.8, 154.0)
- moved C28 128.1 mm to (-589.5, 133.6), turned to -90 degrees
- moved J8 123.5 mm to (-576.0, 130.1)
- moved R9 120.3 mm to (-584.5, 121.8), turned to -90 degrees
- moved C26 120.1 mm to (-585.0, 130.1), turned to -90 degrees
- moved R10 120.1 mm to (-588.5, 121.8), turned to -90 degrees
- moved C27 117.8 mm to (-580.5, 130.1), turned to -90 degrees
- moved D5 113.1 mm to (-584.0, 118.5), turned to 90 degrees
- moved C29 112.9 mm to (-593.7, 140.0)
- moved R5 111.6 mm to (-574.3, 127.0), turned to 180 degrees
- moved R6 102.8 mm to (-582.0, 127.0), turned to 90 degrees
- moved D6 101.6 mm to (-590.5, 118.5), turned to 90 degrees
- moved J9 98.9 mm to (-600.4, 125.4)
- moved TP4 89.3 mm to (-579.0, 124.0)
- moved U10 81.3 mm to (-591.1, 128.5)
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- renumbered C29 to C28, C30 to C29, C31 to C30
Connections:
- C28 pad 1: GNDREF -> /Power+IO/serial_3.3
- C28 pad 2: /Power+IO/serial_3.3 -> GNDREF
- C29 pad 1: GNDREF -> /Power+IO/usb+
- C29 pad 2: /Power+IO/usb+ -> GNDREF
- J4 pad 4: tx_a -> /Power+IO/tx_s
- J4 pad 5: /Power+IO/rx_a -> /Power+IO/rx_s
- J9 pad 1: /Power+IO/tx_s -> tx_a
- R5 pad 2: Net-(U10-CBUS0) -> /Power+IO/vbus_sense
- R6 pad 1: Net-(U10-CBUS0) -> /Power+IO/vbus_sense
- TP4 pad 1: Net-(U10-CBUS0) -> /Power+IO/vbus_sense
- U10 pad 14: /Power+IO/tx_led -> /Power+IO/vbus_sense
- U10 pad 15: Net-(U10-CBUS0) -> /Power+IO/tx_led
- U10 pad 16: unconnected-(U10-CBUS3-Pad16) -> /Power+IO/rx_led
- U10 pad 7: /Power+IO/rx_led -> unconnected-(U10-CBUS2-Pad7)
Routing:
- net /Power+IO/serial_3.3: track 0.00 -> 28.7 mm
- net /Power+IO/n7: track 0.00 -> 21.5 mm
- net /Power+IO/vbus_sense: track 0.00 -> 15.8 mm
- net /Power+IO/tx_s: track 0.00 -> 14.6 mm
- net /Power+IO/usb+: track 0.00 -> 9.23 mm
- net /Power+IO/rx_s: track 0.00 -> 7.64 mm
- net /Power+IO/n3: track 25.8 -> 18.5 mm
- net /Power+IO/tx_led: track 0.00 -> 5.07 mm
- net Net-(D6-K): track 0.00 -> 4.11 mm
- net GNDREF: track 0.00 -> 2.61 mm, vias 0 -> 2
- net /Power+IO/n1: track 7.26 -> 5.02 mm
- net /Power+IO/rx_led: track 0.00 -> 1.95 mm
- net /Power+IO/n4: track 11.1 -> 11.8 mm
Other:
- board text added: "A"
- board text added: "B"
- board text added: "RX"
- board text added: "TX"

Commit message: Set Serial circuit into place
Parts:
- moved C3 92.0 mm to (-593.1, 160.5), turned to 90 degrees
- moved R1 91.0 mm to (-588.0, 160.5), turned to 90 degrees
- moved U9 41.1 mm to (-469.0, 214.9)
- moved Q2 40.1 mm to (-469.0, 207.9)
- moved R4 28.6 mm to (-504.4, 130.0)
- moved U11 28.6 mm to (-504.0, 133.0)
- moved U2 28.6 mm to (-481.2, 81.5)
- moved X1 28.6 mm to (-505.3, 110.0)
- moved C10 28.6 mm to (-484.2, 102.0)
- moved C11 28.6 mm to (-488.7, 102.0)
- moved C12 28.6 mm to (-471.2, 73.7)
- moved C13 28.6 mm to (-475.7, 73.7)
- moved C14 28.6 mm to (-468.2, 89.5)
- moved C15 28.6 mm to (-468.2, 94.0)
- moved C6 28.6 mm to (-503.2, 123.0)
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Routing:
- net /Power+IO/vin: track 0.00 -> 26.6 mm
- net /Power+IO/usb-: track 0.00 -> 25.4 mm
- net /Power+IO/usb+: track 9.23 -> 21.0 mm
- net /Power+IO/rx_s: track 7.64 -> 18.4 mm
- net +5V: track 74.4 -> 81.4 mm
- net /Power+IO/tx_s: track 14.6 -> 17.8 mm
- net /Power+IO/n4: track 11.8 -> 10.6 mm
- net /Power+IO/serial_3.3: track 28.7 -> 29.5 mm

Commit message: Finish power and IO circuit
Parts:
- moved D2 155.4 mm to (-583.5, 155.2), turned to -90 degrees
- moved C2 141.1 mm to (-558.5, 156.5), turned to -90 degrees
- moved D4 138.8 mm to (-550.5, 157.5), turned to 180 degrees
- moved TP2 136.1 mm to (-554.0, 145.5)
- moved Q2 136.0 mm to (-592.5, 151.0)
- moved R8 128.6 mm to (-553.0, 164.5)
- moved U9 108.3 mm to (-556.5, 151.0)
- moved R7 105.2 mm to (-575.0, 156.5), turned to -90 degrees
- moved Q1 99.8 mm to (-580.5, 151.0)
- moved U8 94.8 mm to (-568.5, 151.0)
- moved C1 89.5 mm to (-563.4, 156.5), turned to -90 degrees
- moved D3 83.1 mm to (-570.5, 157.5)
- moved TP1 77.3 mm to (-566.0, 145.5)
- moved C3 1.53 mm to (-593.1, 159.0)
- moved R1 1.28 mm to (-588.0, 159.2)
Routing:
- net /Power+IO/vbus: track 0.00 -> 45.7 mm
- net /Power+IO/n5: track 0.00 -> 40.3 mm
- net +3.3V: track 60.5 -> 84.8 mm
- net +5V: track 81.4 -> 102.0 mm
- net Net-(D4-K): track 0.00 -> 8.05 mm
- net /Power+IO/vin: track 26.6 -> 31.9 mm
- net Net-(D3-K): track 0.00 -> 4.87 mm
- added copper zone on F.Cu, net /Power+IO/vin
Other:
- board text added: "3.3V"
- board text added: "5V"
- board text added: "CAUTION! DO NOT SHORT SINKS"
- board text added: "⚠"

Commit message: Begin final PCB placement
Parts:
- removed the R6 at (-589.1, 132.5)
- added R2: 27, Resistor_THT:R_Axial_DIN0204_L3.6mm_D1.6mm_P2.54mm_Vertical, F.Cu at (-606.8, 142.0)
- added R3: 27, Resistor_THT:R_Axial_DIN0204_L3.6mm_D1.6mm_P2.54mm_Vertical, F.Cu at (-599.2, 145.5)
- added R7: 10k, Resistor_THT:R_Axial_DIN0204_L3.6mm_D1.6mm_P2.54mm_Vertical, F.Cu at (-576.5, 138.7)
- added TP5: ~{AS}, TestPoint:TestPoint_Keystone_5000-5004_Miniature, F.Cu at (-421.2, 88.7)
- added TP6: ~{DTACK}, TestPoint:TestPoint_Keystone_5000-5004_Miniature, F.Cu at (-418.9, 101.5)
- moved C20 191.8 mm to (-534.8, 146.0), turned to 90 degrees
- moved U5 181.1 mm to (-532.4, 157.0), turned to 90 degrees
- moved C21 178.6 mm to (-530.3, 146.0), turned to 90 degrees
- moved U4 167.7 mm to (-532.4, 175.8), turned to 90 degrees
- moved C19 161.0 mm to (-530.0, 164.8), turned to 90 degrees
- moved C18 157.7 mm to (-534.5, 164.8), turned to 90 degrees
- moved C16 124.2 mm to (-590.8, 70.0)
- moved TP3 117.6 mm to (-385.3, 107.2), turned to 90 degrees
- moved SW1 116.6 mm to (-393.3, 117.7), turned to 0 degrees
- moved U11 115.1 mm to (-390.8, 112.5), turned to 0 degrees
- moved C17 113.6 mm to (-590.8, 74.5)
- moved R5 111.9 mm to (-393.8, 112.9), turned to 90 degrees
- moved R4 108.3 mm to (-398.8, 115.2), turned to 0 degrees
- moved C5 108.2 mm to (-393.0, 107.2), turned to 0 degrees
- moved C6 103.0 mm to (-400.8, 111.7), turned to 0 degrees
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- renumbered R9 to R10, R10 to R11, R3 to R4, R4 to R5, R5 to R6, R7 to R8, R8 to R9
Connections:
- J4 pad 4: /Power+IO/tx_s -> /Power+IO/rx_s
- J4 pad 5: /Power+IO/rx_s -> /Power+IO/tx_s
- J9 pad 2: /Power+IO/tx_s -> /Power+IO/rx_s
- J9 pad 4: /Power+IO/tx_s -> /Power+IO/rx_s
- J9 pad 6: /Power+IO/rx_s -> /Power+IO/tx_s
- J9 pad 8: /Power+IO/rx_s -> /Power+IO/tx_s
- U10 pad 8: /Power+IO/usb+ -> Net-(U10-USBDP)
- U10 pad 9: /Power+IO/usb- -> Net-(U10-USBDM)
Routing:
- net +5V: track 102.0 -> 217.3 mm
- net +3.3V: track 84.8 -> 138.9 mm
- net rx_b: track 0.00 -> 50.5 mm
- net rx_a: track 0.00 -> 50.2 mm
- net tx_b: track 0.00 -> 43.5 mm, vias 0 -> 1
- net tx_a: track 0.00 -> 38.9 mm
- net /Memory+Peripheral/po_0: track 0.00 -> 25.5 mm
- net /Memory+Peripheral/pi_0: track 0.00 -> 24.6 mm
- net /Memory+Peripheral/po_2: track 0.00 -> 24.4 mm
- net /Memory+Peripheral/pi_4: track 0.00 -> 23.7 mm
- net /Memory+Peripheral/pi_2: track 0.00 -> 23.7 mm
- net /Memory+Peripheral/pi_5: track 0.00 -> 23.7 mm
- net /Memory+Peripheral/po_4: track 0.00 -> 23.4 mm
- net /Memory+Peripheral/po_6: track 0.00 -> 22.3 mm
- net /Memory+Peripheral/pi_1: track 0.00 -> 15.3 mm
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Other:
- board size 185.3 x 118.5 mm -> 139.7 x 114.3 mm
- board text added: "4.5x5.5{dblquote}"
- board text added: "⌱"
