File: 11x17 Schematic/11x17 Schematic.kicad_sch (KiCad schematic)
At the start: 81 parts, among them J1 Conn_01x06_Pin, J2 Conn_01x03_Pin, J3 Conn_01x08_Pin, J4 Conn_01x06_Pin, J5 Conn_01x02_Pin, J6 Conn_02x04_Odd_Even, J7 USB_B, J8 Conn_01x02_Pin, J9 Conn_01x06_Pin, Q1 AOI21357, Q2 AOI21357, SW1 RESET, U1 XC9572XL, U10 FT230XS, U11 LD1117AV33, U2 MC34064P, U3 MC68000FN, U4 MCM6206CP, U5 28C256, U6 28C256, U7 MCM6206CP, U8 68681, U9 LM7805_TO220, X1 SG-531, X2 EC11

Commit message: Begin monitor development
Parts:
- removed C1, C10, C27, C3, C5, C6, C8: 0.1u, Capacitor_THT:CP_Disc_L5.50mm_W4.00mm_P2.50mm_NonPolarized, symbol Device:C
- removed C11, C13, C15, C17, C19, C2, C21, C28, C4, C7, C9: 1u, Capacitor_THT:CP_Disc_L5.50mm_W4.00mm_P2.50mm_NonPolarized, symbol Device:C
- removed C12, C14, C16, C18, C20, C22: .1u, Capacitor_THT:CP_Disc_L5.50mm_W4.00mm_P2.50mm_NonPolarized, symbol Device:C
- removed C23, C25: 47p, Capacitor_THT:CP_Disc_L5.50mm_W4.00mm_P2.50mm_NonPolarized, symbol Device:C
- removed C24, C26, C29: 4.7u, Capacitor_THT:CP_Radial_D4.0mm_P2.00mm, symbol Device:C_Polarized_US
- removed C30: 10n, Capacitor_THT:CP_Disc_L5.50mm_W4.00mm_P2.50mm_NonPolarized, symbol Device:C
- removed D1, D3, D4, D5: LED, LED_THT:LED_D5.0mm, symbol Device:LED
- removed D2, D6: 1N4001, Diode_THT:D_DO-41_SOD81_P5.08mm_Vertical_KathodeUp, symbol Diode:1N4933-T
- removed F1, F2: 250mA Fuse, Fuse:Fuseholder_Clip-5x20mm_Bel_FC-203-22_Lateral_P17.80x5.00mm_D1.17mm_Horizontal, symbol Device:Fuse
- removed FB1: FerriteBead, Capacitor_THT:C_Axial_L3.8mm_D2.6mm_P10.00mm_Horizontal, symbol Device:FerriteBead
- removed J1, J4, J9: Conn_01x06_Pin, Connector_PinHeader_2.54mm:PinHeader_1x06_P2.54mm_Vertical, symbol Connector:Conn_01x06_Pin
- removed J2: Conn_01x03_Pin, Connector_PinHeader_2.54mm:PinHeader_1x03_P2.54mm_Vertical, symbol Connector:Conn_01x03_Pin
- removed J3: Conn_01x08_Pin, Connector_PinHeader_2.54mm:PinHeader_1x08_P2.54mm_Vertical, symbol Connector:Conn_01x08_Pin
- removed J5, J8: Conn_01x02_Pin, Connector_PinHeader_2.54mm:PinHeader_1x02_P2.54mm_Vertical, symbol Connector:Conn_01x02_Pin
- removed J6: Conn_02x04_Odd_Even, Connector_PinHeader_2.54mm:PinHeader_2x04_P2.54mm_Vertical, symbol Connector_Generic:Conn_02x04_Odd_Even
- removed J7: USB_B, Connector_USB:USB_B_OST_USB-B1HSxx_Horizontal, symbol Connector:USB_B
- removed Q1, Q2: AOI21357, Package_TO_SOT_THT:TO-220-3_Vertical, symbol Transistor_FET:AOI21357
- removed R1, R2, R8: 10k, Resistor_THT:R_Axial_DIN0204_L3.6mm_D1.6mm_P2.54mm_Vertical, symbol Device:R
- removed R10, R11, R9: 220, Resistor_THT:R_Axial_DIN0204_L3.6mm_D1.6mm_P2.54mm_Vertical, symbol Device:R
- removed R3, R5: 27, Resistor_THT:R_Axial_DIN0204_L3.6mm_D1.6mm_P2.54mm_Vertical, symbol Device:R
- removed R4: 470, Resistor_THT:R_Axial_DIN0204_L3.6mm_D1.6mm_P2.54mm_Vertical, symbol Device:R
- removed R6: 1M, Resistor_THT:R_Axial_DIN0204_L3.6mm_D1.6mm_P2.54mm_Vertical, symbol Device:R
- removed R7: 5.6k, Resistor_THT:R_Axial_DIN0204_L3.6mm_D1.6mm_P2.54mm_Vertical, symbol Device:R
- removed SW1: RESET, Button_Switch_THT:SW_PUSH_6mm, symbol Switch:SW_Push
- removed TP1: ~{AS}, TestPoint:TestPoint_Keystone_5000-5004_Miniature, symbol Connector:TestPoint
- removed TP2: ~{DTACK}, TestPoint:TestPoint_Keystone_5000-5004_Miniature, symbol Connector:TestPoint
- removed TP3: ~{HLT}/~{RST}, TestPoint:TestPoint_Keystone_5000-5004_Miniature, symbol Connector:TestPoint
- removed TP4: 5V TEST, TestPoint:TestPoint_Keystone_5000-5004_Miniature, symbol Connector:TestPoint
- removed TP5: VBUS SENSE, TestPoint:TestPoint_Keystone_5000-5004_Miniature, symbol Connector:TestPoint
- removed TP6: 3V TEST, TestPoint:TestPoint_Keystone_5000-5004_Miniature, symbol Connector:TestPoint
- removed U1: XC9572XL, Package_LCC:PLCC-44_THT-Socket, symbol CPLD_Xilinx:XC9572XL-PC44
- removed U10: FT230XS, Package_SO:SSOP-16_3.9x4.9mm_P0.635mm, symbol Interface_USB:FT230XS
- removed U11: LD1117AV33, Package_TO_SOT_THT:TO-220-3_Vertical, symbol Regulator_Linear:LD1117-3.3
- removed U2: MC34064P, Package_TO_SOT_THT:TO-92_Inline, symbol Power_Supervisor:MC34064P
- removed U3: MC68000FN, Package_LCC:PLCC-68_THT-Socket, symbol CPU_NXP_68000:MC68000FN
- removed U4, U7: MCM6206CP, Package_DIP:DIP-28_W7.62mm_Socket, symbol Memory_RAM:MCM6206CP
- removed U5, U6: 28C256, Package_DIP:DIP-28_W15.24mm_Socket, symbol Memory_EEPROM:28C256
- removed U8: 68681, Package_DIP:DIP-40_W15.24mm_Socket, symbol Interface:68681
- removed U9: LM7805_TO220, Package_TO_SOT_THT:TO-220-3_Vertical, symbol Regulator_Linear:LM7805_TO220
- removed X1: SG-531, Oscillator:Oscillator_SeikoEpson_SG-8002DC, symbol Oscillator:SG-531
- removed X2: EC11, Oscillator:Oscillator_DIP-8, symbol Oscillator:EC11
- added C31, C33, C35, C37, C39, C41, C43, C52, C61: 0.1u, Capacitor_THT:CP_Disc_L5.50mm_W4.00mm_P2.50mm_NonPolarized, symbol Device:C
- added C32, C34, C36, C38, C40, C42, C45, C47, C49, C51, C53, C55, C62: 1u, Capacitor_THT:CP_Disc_L5.50mm_W4.00mm_P2.50mm_NonPolarized, symbol Device:C
- added C44, C46, C48, C50, C54, C56: .1u, Capacitor_THT:CP_Disc_L5.50mm_W4.00mm_P2.50mm_NonPolarized, symbol Device:C
- added C57, C59: 47p, Capacitor_THT:CP_Disc_L5.50mm_W4.00mm_P2.50mm_NonPolarized, symbol Device:C
- added C58, C60, C63: 4.7u, Capacitor_THT:CP_Radial_D4.0mm_P2.00mm, symbol Device:C_Polarized_US
- added C64: 10n, Capacitor_THT:CP_Disc_L5.50mm_W4.00mm_P2.50mm_NonPolarized, symbol Device:C
- added D10, D12: 1N4001, Diode_THT:D_DO-41_SOD81_P5.08mm_Vertical_KathodeUp, symbol Diode:1N4933-T
- added D11, D7, D8, D9: LED, LED_THT:LED_D5.0mm, symbol Device:LED
- added F3, F4: 250mA Fuse, Fuse:Fuseholder_Clip-5x20mm_Bel_FC-203-22_Lateral_P17.80x5.00mm_D1.17mm_Horizontal, symbol Device:Fuse
- added FB2: FerriteBead, Capacitor_THT:C_Axial_L3.8mm_D2.6mm_P10.00mm_Horizontal, symbol Device:FerriteBead
- added J10, J13, J18: Conn_01x06_Pin, Connector_PinHeader_2.54mm:PinHeader_1x06_P2.54mm_Vertical, symbol Connector:Conn_01x06_Pin
- added J11: Conn_01x03_Pin, Connector_PinHeader_2.54mm:PinHeader_1x03_P2.54mm_Vertical, symbol Connector:Conn_01x03_Pin
- added J12: Conn_01x08_Pin, Connector_PinHeader_2.54mm:PinHeader_1x08_P2.54mm_Vertical, symbol Connector:Conn_01x08_Pin
- added J14, J17: Conn_01x02_Pin, Connector_PinHeader_2.54mm:PinHeader_1x02_P2.54mm_Vertical, symbol Connector:Conn_01x02_Pin
- added J15: Conn_02x04_Odd_Even, Connector_PinHeader_2.54mm:PinHeader_2x04_P2.54mm_Vertical, symbol Connector_Generic:Conn_02x04_Odd_Even
- added J16: USB_B, Connector_USB:USB_B_OST_USB-B1HSxx_Horizontal, symbol Connector:USB_B
- added Q3, Q4: AOI21357, Package_TO_SOT_THT:TO-220-3_Vertical, symbol Transistor_FET:AOI21357
- added R12, R13, R14, R15, R23: 10k, Resistor_THT:R_Axial_DIN0204_L3.6mm_D1.6mm_P2.54mm_Vertical, symbol Device:R
- added R16, R17, R24: 220, Resistor_THT:R_Axial_DIN0204_L3.6mm_D1.6mm_P2.54mm_Vertical, symbol Device:R
- added R18, R20: 27, Resistor_THT:R_Axial_DIN0204_L3.6mm_D1.6mm_P2.54mm_Vertical, symbol Device:R
- added R19: 470, Resistor_THT:R_Axial_DIN0204_L3.6mm_D1.6mm_P2.54mm_Vertical, symbol Device:R
- added R21: 1M, Resistor_THT:R_Axial_DIN0204_L3.6mm_D1.6mm_P2.54mm_Vertical, symbol Device:R
- added R22: 5.6k, Resistor_THT:R_Axial_DIN0204_L3.6mm_D1.6mm_P2.54mm_Vertical, symbol Device:R
- added SW2: RESET, Button_Switch_THT:SW_PUSH_6mm, symbol Switch:SW_Push
- added TP10: ~{RST}, TestPoint:TestPoint_Keystone_5000-5004_Miniature, symbol Connector:TestPoint
- added TP11: 5V TEST, TestPoint:TestPoint_Keystone_5000-5004_Miniature, symbol Connector:TestPoint
- added TP12: 3.3V TEST, TestPoint:TestPoint_Keystone_5000-5004_Miniature, symbol Connector:TestPoint
- added TP13: VBUS SENSE, TestPoint:TestPoint_Keystone_5000-5004_Miniature, symbol Connector:TestPoint
- added TP14: GND POINT, TestPoint:TestPoint_Keystone_5000-5004_Miniature, symbol Connector:TestPoint
- added TP7: ~{AS}, TestPoint:TestPoint_Keystone_5000-5004_Miniature, symbol Connector:TestPoint
- added TP8: ~{DTACK}, TestPoint:TestPoint_Keystone_5000-5004_Miniature, symbol Connector:TestPoint
- added TP9: ~{BERR}, TestPoint:TestPoint_Keystone_5000-5004_Miniature, symbol Connector:TestPoint
- added U12: MC68000FN, Package_LCC:PLCC-68_THT-Socket, symbol CPU_NXP_68000:MC68000FN
- added U13: XC9572XL, Package_LCC:PLCC-44_THT-Socket, symbol CPLD_Xilinx:XC9572XL-PC44
- added U14: MC34064P, Package_TO_SOT_THT:TO-92_Inline, symbol Power_Supervisor:MC34064P
- added U15, U17: MCM6206CP, Package_DIP:DIP-28_W7.62mm_Socket, symbol Memory_RAM:MCM6206CP
- added U16, U18: 28C256, Package_DIP:DIP-28_W15.24mm_Socket, symbol Memory_EEPROM:28C256
- added U19: 68681, Package_DIP:DIP-40_W15.24mm_Socket, symbol Interface:68681
- added U20: LM7805_TO220, Package_TO_SOT_THT:TO-220-3_Vertical, symbol Regulator_Linear:LM7805_TO220
- added U21: FT230XS, Package_SO:SSOP-16_3.9x4.9mm_P0.635mm, symbol Interface_USB:FT230XS
- added U22: LD1117AV33, Package_TO_SOT_THT:TO-220-3_Vertical, symbol Regulator_Linear:LD1117-3.3
- added X3: SG-531, Oscillator:Oscillator_SeikoEpson_SG-8002DC, symbol Oscillator:SG-531
- added X4: EC11, Oscillator:Oscillator_DIP-8, symbol Oscillator:EC11
Connections:
- net +3.3V: now also C37.1, C38.1, C39.1, C40.1, C41.1, C42.1, C63.1, D11.2 (A), J10.6 (Pin_6), J11.3 (Pin_3), R12.1, TP12.1, U13.21 (V_{cc-INT}-3.3V), U13.32 (V_{cc-IO}-3.3V), U13.41 (V_{cc-INT}-3.3V), U22.2 (VO)
- net +5V: now also C31.1, C32.1, C33.1, C34.1, C35.1, C36.1, C44.1, C45.1, C46.1, C47.1, C48.1, C49.1, C50.1, C51.1, C52.1, C53.1, C54.1, C55.1, C58.1, D9.2 (A), J11.1 (Pin_1), J14.2 (Pin_2), J18.3 (Pin_3), Q3.3 (S), R13.1, R15.1, TP11.1, U12.12 (~{BGACK}), U12.13 (~{BR}), U12.14 (VCC), U12.23 (~{VPA}), U12.52 (VCC), U15.28 (VCC), U16.28 (VCC), U17.28 (VCC), U18.28 (VCC), U19.40 (VCC), U20.3 (VO), X3.1 (OE), X3.8 (Vcc), X4.1 (OE), X4.8 (Vcc)
- net GNDREF: now also C31.2, C32.2, C33.2, C34.2, C35.2, C36.2, C37.2, C38.2, C39.2, C40.2, C41.2, C42.2, C43.2, C44.2, C45.2, C46.2, C47.2, C48.2, C49.2, C50.2, C51.2, C52.2, C53.2, C54.2, C55.2, C56.2, C57.2, C58.2, C59.2, C60.2, C61.2, C62.2, C63.2, C64.2, J10.5 (Pin_5), J11.2 (Pin_2), J16.4 (GND), J17.2 (Pin_2), J18.1 (Pin_1), R14.1, R19.2, R21.2, R23.1, R24.2, TP14.1, U12.16 (GND), U12.17 (GND), U12.56 (GND), U12.57 (GND), U13.10 (GND), U13.23 (GND), U13.31 (GND), U14.3 (GND), U15.14 (GND), U16.14 (GND), U17.14 (GND), U18.14 (GND), U19.20 (GND), U19.33 (X2), U20.2 (GND), U21.13 (GND), U21.5 (GND), U22.1 (GND), X3.4 (GND), X4.4 (GND)
- net addr0: now also U12.32 (A1), U15.9 (A1), U16.10 (A0), U17.9 (A1), U18.10 (A0), U19.1 (RS1)
- net addr1: now also U12.33 (A2), U15.7 (A3), U16.9 (A1), U17.7 (A3), U18.9 (A1), U19.3 (RS2)
- net addr10: now also U12.42 (A11), U15.23 (A11), U16.21 (A10), U17.23 (A11), U18.21 (A10)
- net addr11: now also U12.43 (A12), U15.24 (A9), U16.23 (A11), U17.24 (A9), U18.23 (A11)
- net addr12: now also U12.44 (A13), U15.26 (A13), U16.2 (A12), U17.26 (A13), U18.2 (A12)
- net addr13: now also U12.45 (A14), U15.25 (A8), U16.26 (A13), U17.25 (A8), U18.26 (A13)
- net addr14: now also U12.46 (A15), U15.10 (A0), U16.1 (A14), U17.10 (A0), U18.1 (A14)
- net addr15: now also U12.47 (A16), U13.39 (P39/GSR)
- net addr16: now also U12.48 (A17), U13.37 (P37)
- net addr17: now also U12.49 (A18), U13.38 (P38)
- net addr18: now also U12.50 (A19), U13.35 (P35)
- net addr19: now also U12.51 (A20), U13.36 (P36)
- net addr2: now also U12.34 (A3), U15.8 (A2), U16.8 (A2), U17.8 (A2), U18.8 (A2), U19.5 (RS3)
- net addr20: now also U12.53 (A21), U13.33 (P33)
- net addr21: now also U12.54 (A22), U13.29 (P29)
- net addr22: now also U12.55 (A23), U13.34 (P34)
- net addr3: now also U12.35 (A4), U15.5 (A5), U16.7 (A3), U17.5 (A5), U18.7 (A3), U19.6 (RS4)
- net addr4: now also U12.36 (A5), U15.6 (A4), U16.6 (A4), U17.6 (A4), U18.6 (A4)
- net addr5: now also U12.37 (A6), U15.1 (A14), U16.5 (A5), U17.1 (A14), U18.5 (A5)
- net addr6: now also U12.38 (A7), U15.4 (A6), U16.4 (A6), U17.4 (A6), U18.4 (A6)
- net addr7: now also U12.39 (A8), U15.3 (A7), U16.3 (A7), U17.3 (A7), U18.3 (A7)
- net addr8: now also U12.40 (A9), U15.2 (A12), U16.25 (A8), U17.2 (A12), U18.25 (A8)
- net addr9: now also U12.41 (A10), U15.21 (A10), U16.24 (A9), U17.21 (A10), U18.24 (A9)
- net as: now also TP7.1, U12.6 (~{AS}), U13.28 (P28)
- net berr: now also TP9.1, U12.24 (~{BERR}), U13.18 (P18)
- net clk: now also U12.15 (CLK), U13.5 (P5/GCK1), X3.5 (OUT)
- net data0: now also U12.5 (D0), U15.11 (Q0), U16.11 (D0), U19.25 (D0)
- net data1: now also U12.4 (D1), U15.12 (Q1), U16.12 (D1), U19.16 (D1)
- net data10: now also U12.63 (D10), U17.18 (Q6), U18.13 (D2)
- net data11: now also U12.62 (D11), U17.17 (Q5), U18.15 (D3)
- net data12: now also U12.61 (D12), U17.16 (Q4), U18.16 (D4)
- net data13: now also U12.60 (D13), U17.15 (Q3), U18.17 (D5)
- net data14: now also U12.59 (D14), U17.12 (Q1), U18.18 (D6)
- net data15: now also U12.58 (D15), U17.11 (Q0), U18.19 (D7)
- net data2: now also U12.3 (D2), U15.13 (Q2), U16.13 (D2), U19.24 (D2)
- net data3: now also U12.2 (D3), U15.19 (Q7), U16.15 (D3), U19.17 (D3)
- net data4: now also U12.1 (D4), U15.18 (Q6), U16.16 (D4), U19.23 (D4)
- net data5: now also U12.68 (D5), U15.17 (Q5), U16.17 (D5), U19.18 (D5)
- net data6: now also U12.67 (D6), U15.16 (Q4), U16.18 (D6), U19.22 (D6)
- net data7: now also U12.66 (D7), U15.15 (Q3), U16.19 (D7), U19.19 (D7)
- net data8: now also U12.65 (D8), U17.13 (Q2), U18.11 (D0)
- net data9: now also U12.64 (D9), U17.19 (Q7), U18.12 (D1)
- net dtack: now also TP8.1, U12.10 (~{DTACK}), U13.24 (P24)
- net duart_cs: now also U13.1 (P1), U19.35 (CS)
- net duart_dtack: now also U13.2 (P2), U19.9 (~{DTACK})
- net duart_iack: now also U13.42 (P42/GTS1), U19.37 (~{IACK})
- net duart_irq: now also U13.4 (P4), U19.21 (~{IRQ})
- net duart_rw: now also U13.3 (P3), U19.8 (R/W)
- net fc0: now also U12.30 (FC0), U13.19 (P19)
- net fc1: now also U12.29 (FC1), U13.11 (P11)
- net fc2: now also U12.28 (FC2), U13.13 (P13)
- net ipl0: now also U12.27 (~{IPL0}), U13.12 (P12)
- net ipl1: now also U12.26 (~{IPL1}), U13.14 (P14)
- net ipl2: now also U12.25 (~{IPL2}), U13.20 (P20)
- net lds: now also U12.8 (~{LDS}), U13.26 (P26)
- net n1: now also D12.2 (A), J17.1 (Pin_1)
- net n2: now also D12.1 (K), F4.2
- net n3: now also C64.1, F3.1, J16.1 (VBUS)
- net n4: now also F3.2, FB2.1
- net n5: now also D10.1 (K), Q4.3 (S), U22.3 (VI)
- net n6: now also R13.2, SW2.1, U14.2 (IN)
- net n7: now also C61.1, C62.1, J14.1 (Pin_1), U21.12 (VCC)
- net oe: now also U13.6 (P6/GCK2), U15.22 (~{OE}), U16.22 (~{OE}), U17.22 (~{OE}), U18.22 (~{OE})
- net pi_0: now also J13.1 (Pin_1), U19.7 (IP0)
- net pi_1: now also J13.2 (Pin_2), U19.4 (IP1)
- net pi_2: now also J13.3 (Pin_3), U19.36 (IP2)
- net pi_3: now also J13.4 (Pin_4), U19.2 (IP3)
- net pi_4: now also J13.5 (Pin_5), U19.39 (IP4)
- net pi_5: now also J13.6 (Pin_6), U19.38 (IP5)
- net po_0: now also J12.1 (Pin_1), U19.29 (OP0)
- net po_1: now also J12.2 (Pin_2), U19.12 (OP1)
- net po_2: now also J12.3 (Pin_3), U19.28 (OP2)
- net po_3: now also J12.4 (Pin_4), U19.13 (OP3)
- net po_4: now also J12.5 (Pin_5), U19.27 (OP4)
- net po_5: now also J12.6 (Pin_6), U19.14 (OP5)
- net po_6: now also J12.7 (Pin_7), U19.26 (OP6)
- net po_7: now also J12.8 (Pin_8), U19.15 (OP7)
- net ramh_cs: now also U13.8 (P8), U17.20 (~{CS})
- net raml_cs: now also U13.9 (P9), U15.20 (~{CS})
- net romh_cs: now also U13.43 (P43), U18.20 (~{CS})
- net roml_cs: now also U13.40 (P40/GTS2), U16.20 (~{CS})
- net rw: now also U12.9 (~{R/W}), U13.25 (P25)
- net rx_a: now also J15.1 (Pin_1), U19.31 (RXDA)
- net rx_b: now also J15.3 (Pin_3), U19.10 (RXDB)
- net rx_led: now also R17.2, U21.16 (CBUS3)
- net rx_s: now also J15.6 (Pin_6), J15.8 (Pin_8), J18.4 (Pin_4), U21.4 (RXD)
- net serial_3.3: now also C56.1, D7.2 (A), D8.2 (A), U21.10 (3V3OUT), U21.3 (VCCIO)
- net tck: now also J10.4 (Pin_4), U13.17 (TCK)
- net tdi: now also J10.2 (Pin_2), U13.15 (TDI)
- net tdo: now also J10.3 (Pin_3), U13.30 (TDO)
- net tms: now also J10.1 (Pin_1), U13.16 (TMS)
- net tx_a: now also J15.5 (Pin_5), U19.30 (TXDA)
- net tx_b: now also J15.7 (Pin_7), U19.11 (TXDB)
- net tx_led: now also R16.2, U21.15 (CBUS0)
- net tx_s: now also J15.2 (Pin_2), J15.4 (Pin_4), J18.5 (Pin_5), U21.1 (TXD)
- net uds: now also U12.7 (~{UDS}), U13.27 (P27)
- net usb+: now also C57.1, J16.3 (D+), R18.1
- net usb-: now also C59.1, J16.2 (D-), R20.1
- net vbus: now also FB2.2, Q3.2 (D), Q4.2 (D), R22.1
- net vbus_sense: now also R22.2, R23.2, TP13.1, U21.14 (CBUS1)
- net vin: now also C60.1, D10.2 (A), F4.1, Q3.1 (G), Q4.1 (G), R21.1, U20.1 (VI)
- net we: now also U13.7 (P7/GCK3), U15.27 (~{WE}), U16.27 (~{WE}), U17.27 (~{WE}), U18.27 (~{WE})
- new net: D8.1 (K), R17.1
- new net: D7.1 (K), R16.1
- new net: D11.1 (K), R24.1
- new net: D9.1 (K), R19.1
- new net duart_clk: U19.32 (X1/CLK), X4.5 (OUT)
- new net hlt: R12.2, U12.19 (~{HALT}), U13.22 (P22)
- new net n10: R14.2, R20.2, SW2.2, U21.9 (USBDM)
- new net n9: R18.2, U21.8 (USBDP)
- new net rst: C43.1, R15.2, TP10.1, U12.20 (~{RESET}), U13.44 (P44), U14.1 (~{RESET}), U19.34 (~{RESET}), U21.11 (~{RESET})
- no-connect marks 10 -> 9
Other:
- note added: "RANDOM ACCESS"
- note added: "READ ONLY"
- note removed: "GCK=Global clock GTS=Global output enable GSR=Global set/reset CPLD control signals GTS 1 and 2 do the same thing"
- note removed: "RANDOM ACCESS MEMORY"
- note removed: "READ ONLY MEMORY"
